File: hardware/if-9mhz.sch (KiCad schematic (older format))
At the start: 29 parts, among them Q13 MMBT3904, T4 FT37-43, U7 ADE-6, Y1 9Mhz, Y2 9Mhz, Y3 9Mhz, Y4 9Mhz, Y5 9Mhz

Commit message: Clarify that second IF can be other than 9 Mhz
Other:
- note added: "Xtals should be measured using G3UUR method,\nand suitable capacitors should be picked in LTspice.\nXtals should be matched by the resonant frequency.\n\nIt’s possible to use xtals for another frequency. Only\na slight change of the firmware is required in this case,\nand maybe a little adjustment of the AGC circuit.\nAnother number of xtals can be used as well.\n\nhttps://eax.me/crystal-measurem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"
- note removed: "Xtals should be measured using G3UUR method,\nand suitable capacitors should be picked in LTspice.\nXtals should be matched by the resonant frequency.\n\nhttps://eax.me/crystal-measurements/\nhttps://eax.me/crystal-filters-part-4/"
Changed lines of the file:
@@
 	-1   0    0    1
 $EndComp
-Text Notes 5100 6400 0    50   ~ 0
-Xtals should be measured using G3UUR method,\nand suitable capacitors should be picked in LTspice.\nXtals should be matched by the resonant frequency.\n\nhttps://eax.me/crystal-measurements/\nhttps://eax.me/crystal-filters-part-4/
+Text Notes 5100 6800 0    50   ~ 0
+Xtals should be measured using G3UUR method,\nand suitable capacitors should be picked in LTspice.\nXtals should be matched by the resonant frequency.\n\nIt’s possible to use xtals for another frequency. Only\na slight change of the firmware is required in this case,\nand maybe a little adjustment of the AGC circuit.\nAnother number of xtals can be used as well.\n\nhttps://eax.me/crystal-measurements/\nhttps://eax.me/crystal-filters-part-4/
 $EndSCHEMATC
