File: hardware/hbr-cw.kicad_pcb (KiCad board)
At the start: 2 copper layers, 153.7 x 185.4 mm, 411 parts, among them J1 ON/OFF, J10 BluePill_Right, J11 MAIN, J12 BAND, J13 LCD 0802, J14 RIT/XIT, J15 FAST, J16 LOCK, J17 RFAMP, J18 CLAR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

Commit message: Update the silkscreen a little
Other:
- board text added: "HBR/CW by Alex R2AUK, Jan 2022 https://github.com/afiskon/hbr-cw"
- board text removed: "HBR/CW by Alex R2AUK, 2022 https://eax.me/hbr-cw-pcb/"

Commit message: Add a warning that U1 can get a little hot + minor changes
Other:
- board text added: "GETS HOT"
